File: 24V Fixture Board/24V Fixture Board.kicad_sch (KiCad schematic)
At the start: 6 parts, among them J1 LED_IN, J2 Conn_01x03

Commit message: Add BOM
Parts:
- C1: value 1000u -> 1μF; footprint (none) -> Capacitor_THT:CP_Radial_D4.0mm_P2.00mm
- J1: footprint (none) -> TerminalBlock_MetzConnect:TerminalBlock_MetzConnect_Type011_RT05504HBWC_1x04_P5.00mm_Horizontal
- U1: footprint (none) -> LM2596S-Buck-Module:LM2596S-Buck-Module
- U2: footprint (none) -> Max485:Max485
Changed lines of the file:
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@@
 			)
 		)
-		(property "Footprint" ""
+		(property "Footprint" "LM2596S-Buck-Module:LM2596S-Buck-Module"
 			(at 174.752 26.924 0)
 			(effects
@@
 			)
 		)
-		(property "Footprint" ""
+		(property "Footprint" "TerminalBlock_MetzConnect:TerminalBlock_MetzConnect_Type011_RT05504HBWC_1x04_P5.00mm_Horizontal"
 			(at 269.24 31.75 0)
 			(effects
@@
 			)
 		)
-		(property "Footprint" ""
+		(property "Footprint" "Max485:Max485"
 			(at 173.99 67.31 0)
 			(effects
@@
 			)
 		)
-		(property "Value" "1000u"
+		(property "Value" "1μF"
 			(at 157.48 33.4009 0)
 			(effects
@@
 			)
 		)
-		(property "Footprint" ""
+		(property "Footprint" "Capacitor_THT:CP_Radial_D4.0mm_P2.00mm"
 			(at 154.6352 36.83 0)
 			(effects
