File: 24V Fixture Board/24V Fixture Board.kicad_pcb (KiCad board)
At the start: 2 copper layers, 23 x 68.4 mm, 6 parts, among them J1 LED_IN, J2 Conn_01x03

Commit message: 27th Mega Commit
Routing:
- net LED-: track 65.8 -> 33.5 mm
- net +24V: track 88.5 -> 74.1 mm
- net GND: track 90.3 -> 77.9 mm
- net +5V: track 40.5 -> 44.6 mm
