File: DMX Control Board/DMX Control Board.kicad_pcb (KiCad board)
At the start: 2 copper layers, 133 x 91 mm, 32 parts, among them J1 DC_IN, J2 DMX_IN, J3 LED1, J4 LED2, J5 LED3, J6 LED4, U1 ESP32-DevKitC_Headers

Commit message: The Great Fixit
Parts:
- F1, F2, F3, F4: footprint Fuse:Fuseholder_Blade_Mini_Keystone_3568 -> Fuse:FuseHolder_Blade_ATO_Littelfuse_FLR_178.6165
- moved F1 2.94 mm to (192.1, 98.0)
- moved F2 2.94 mm to (192.1, 105.3)
- moved F4 2.94 mm to (192.2, 119.9)
- moved F3 2.94 mm to (192.1, 112.6)
Routing:
- net Net-(J3-Pin_1): track 123.2 -> 177.0 mm, vias 2 -> 1
- net +5V: track 295.0 -> 253.3 mm, vias 2 -> 0
- net DMXIN-: track 28.2 -> 55.8 mm
- net Net-(J4-Pin_1): track 94.1 -> 116.3 mm, vias 2 -> 0
- net Net-(J5-Pin_1): track 67.5 -> 82.6 mm, vias 2 -> 0
- net WLED4: track 58.6 -> 48.3 mm
- net LED4+: track 25.7 -> 18.8 mm, vias 2 -> 0
- net +24V: track 142.5 -> 137.1 mm, vias 1 -> 0
- net LED3+: track 24.5 -> 19.7 mm, vias 1 -> 0
- net LED2+: track 24.5 -> 19.7 mm, vias 2 -> 0
- net LED1+: track 24.5 -> 19.7 mm, vias 2 -> 0
- net LED1-: track 22.4 -> 27.0 mm, vias 2 -> 0
- net LED2-: track 22.3 -> 26.7 mm, vias 2 -> 0
- net LED3-: track 22.3 -> 26.6 mm, vias 1 -> 0
- net WLED1: track 26.3 -> 30.0 mm
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