File: DMX Control Board/DMX Control Board.kicad_sch (KiCad schematic)
At the start: 31 parts, among them J1 DC_IN, J2 DMX_IN, J3 LED1, J4 LED2, J5 LED3, J6 LED4, U1 ESP32-DevKitC_Headers

Commit message: The Great Fixit
Parts:
- F1, F2, F3, F4: footprint Fuse:Fuseholder_Blade_Mini_Keystone_3568 -> Fuse:FuseHolder_Blade_ATO_Littelfuse_FLR_178.6165
Changed lines of the file:
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@@
 			)
 		)
-		(property "Footprint" "Fuse:Fuseholder_Blade_Mini_Keystone_3568"
+		(property "Footprint" "Fuse:FuseHolder_Blade_ATO_Littelfuse_FLR_178.6165"
 			(at 251.46 46.228 90)
 			(effects
@@
 			)
 		)
-		(property "Footprint" "Fuse:Fuseholder_Blade_Mini_Keystone_3568"
+		(property "Footprint" "Fuse:FuseHolder_Blade_ATO_Littelfuse_FLR_178.6165"
 			(at 251.46 135.128 90)
 			(effects
@@
 			)
 		)
-		(property "Footprint" "Fuse:Fuseholder_Blade_Mini_Keystone_3568"
+		(property "Footprint" "Fuse:FuseHolder_Blade_ATO_Littelfuse_FLR_178.6165"
 			(at 251.46 75.438 90)
 			(effects
@@
 			)
 		)
-		(property "Footprint" "Fuse:Fuseholder_Blade_Mini_Keystone_3568"
+		(property "Footprint" "Fuse:FuseHolder_Blade_ATO_Littelfuse_FLR_178.6165"
 			(at 251.46 104.648 90)
 			(effects

Commit message: 27th Mega Commit
Parts:
- J1: footprint PJ_063AH:CUI_PJ-063AH -> XUNPU:DC-IN-TH_DC-S010A-D025-20A
Changed lines of the file:
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@@
 			)
 		)
-		(property "Footprint" "PJ_063AH:CUI_PJ-063AH"
+		(property "Footprint" "XUNPU:DC-IN-TH_DC-S010A-D025-20A"
 			(at 242.57 27.94 0)
 			(effects
